File: pcbs/amoebae/amoeba-stabilizer-7-promicro.kicad_pcb (KiCad board)
At the start: 2 copper layers, 125.5 x 21.6 mm, 70 parts

Commit message: Fix board outline and SR0 track
Routing:
- net /key/SR0: track 156.8 -> 157.6 mm
Other:
- outline, holes or cut-outs redrawn
Changed lines of the file:
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@@
-(kicad_pcb (version 20171130) (host pcbnew "(5.0.1)-3")
+(kicad_pcb (version 20171130) (host pcbnew "(5.1.5)-3")
   (general
     (thickness 1.6)
-    (drawings 152)
+    (drawings 150)
     (tracks 243)
     (zones 0)
@@
   (page A3)
   (layers
-    (0 F.Cu signal hide)
-    (31 B.Cu signal hide)
-    (32 B.Adhes user hide)
-    (33 F.Adhes user hide)
-    (34 B.Paste user hide)
-    (35 F.Paste user hide)
+    (0 F.Cu signal)
+    (31 B.Cu signal)
+    (32 B.Adhes user)
+    (33 F.Adhes user)
+    (34 B.Paste user)
+    (35 F.Paste user)
     (36 B.SilkS user)
     (37 F.SilkS user)
-    (38 B.Mask user hide)
-    (39 F.Mask user hide)
-    (40 Dwgs.User user hide)
-    (41 Cmts.User user hide)
-    (42 Eco1.User user hide)
-    (43 Eco2.User user hide)
+    (38 B.Mask user)
+    (39 F.Mask user)
+    (40 Dwgs.User user)
+    (41 Cmts.User user)
+    (42 Eco1.User user)
+    (43 Eco2.User user)
     (44 Edge.Cuts user)
   )
@@
     (zone_45_only no)
     (trace_min 0.1524)
-    (segment_width 0.1)
-    (edge_width 0.1)
     (via_size 0.889)
     (via_drill 0.635)
@@
     (uvia_min_size 0.508)
     (uvia_min_drill 0.127)
+    (edge_width 0.1)
+    (segment_width 0.1)
     (pcb_text_width 0.3)
     (pcb_text_size 1.5 1.5)
@@
     (visible_elements 7FFFF7FF)
     (pcbplotparams
-      (layerselection 0x00030_ffffffff)
+      (layerselection 0x000f0_ffffffff)
       (usegerberextensions true)
       (usegerberattributes false)
@@
       (plotinvisibletext false)
       (padsonsilk false)
-      (subtractmaskfromsilk false)
+      (subtractmaskfromsilk true)
       (outputformat 1)
       (mirror false)
       (drillshape 0)
       (scaleselection 1)
-      (outputdirectory "gerber/"))
+      (outputdirectory "gerbers/"))
   )
   (net 0 "")
@@
   (gr_arc (start 196.469 100.218) (end 196.469 100.98) (angle 90) (layer Edge.Cuts) (width 0.1))
   (gr_arc (start 301.371 100.218) (end 302.133 100.218) (angle 90) (layer Edge.Cuts) (width 0.1))
-  (gr_line (start 251.42 105.99) (end 251.46 105.41) (layer Edge.Cuts) (width 0.1))
   (gr_line (start 304.546 117.49) (end 304.546 118.09325) (angle 90) (layer Edge.Cuts) (width 0.1))
   (gr_arc (start 302.9585 118.09325) (end 302.9585 119.68075) (angle -90) (layer Edge.Cuts) (width 0.1))
   (gr_line (start 193.294 117.49) (end 193.294 118.09325) (angle 90) (layer Edge.Cuts) (width 0.1))
   (gr_arc (start 194.8815 118.09325) (end 193.294 118.09325) (angle -90) (layer Edge.Cuts) (width 0.1))
-  (gr_line (start 194.8815 119.68075) (end 302.92675 119.68075) (angle 90) (layer Edge.Cuts) (width 0.1))
+  (gr_line (start 194.8815 119.68075) (end 302.9585 119.68075) (angle 90) (layer Edge.Cuts) (width 0.1))
   (gr_arc (start 304.292 100.218) (end 302.133 100.218) (angle 90) (layer Edge.Cuts) (width 0.1))
   (gr_line (start 304.292 98.059) (end 307.213 98.059) (angle 90) (layer Edge.Cuts) (width 0.1))
@@
     (arrow2b (pts (xy 248.92 82.8675) (xy 247.793496 83.453921)))
   )
-  (gr_line (start 251.42 105.99) (end 251.46 105.41) (angle 90) (layer Edge.Cuts) (width 1.4986))
   (gr_text v1.5 (at 257.3655 115.189) (layer B.SilkS)
     (effects (font (size 0.8 0.8) (thickness 0.15) italic) (justify mirror))
@@
   (segment (start 202.216 118.175) (end 200.6285 116.5875) (width 0.254) (layer F.Cu) (net 4))
   (segment (start 246.253 111.76) (end 246.2276 111.7854) (width 0.254) (layer F.Cu) (net 4))
-  (segment (start 199.83475 107.315) (end 188.4045 107.315) (width 0.254) (layer F.Cu) (net 4))
   (segment (start 246.2276 111.7854) (end 242.7605 111.7854) (width 0.254) (layer F.Cu) (net 4))
   (segment (start 242.7605 111.7854) (end 241.9035 112.6424) (width 0.254) (layer F.Cu) (net 4))
@@
   (segment (start 251.409201 115.285219) (end 251.693982 115.57) (width 0.254) (layer B.Cu) (net 4))
   (segment (start 298.371 108.3) (end 308.4505 108.3) (width 0.254) (layer F.Cu) (net 4))
+  (segment (start 199.83475 107.315) (end 187.61075 107.315) (width 0.254) (layer F.Cu) (net 4))
   (segment (start 243.84 113.03) (end 246.38 113.03) (width 0.254) (layer F.Cu) (net 5))
   (segment (start 246.888 113.538) (end 246.634 113.284) (width 0.254) (layer B.Cu) (net 5))
